File: SRC/GPS_MODULE_V3/GPS_MODULE_V3.kicad_sch (KiCad schematic)
At the start: 11 parts, among them J1 Input, J4 Conn_01x04, Q1 SSM3J328R-HXY

Commit message: layut completed
Parts:
- removed J4: Conn_01x04, symbol Connector_Generic:Conn_01x04
- added J2: Conn_02x02_Odd_Even, Connector_Molex:Molex_Mini-Fit_Jr_5569-04A2_2x02_P4.20mm_Horizontal, symbol Connector_Generic:Conn_02x02_Odd_Even
Connections:
- net +5V: now also J2.2 (Pin_2)
- net GND: now also J2.4 (Pin_4)
- net RS485_MAX485/A: now also J2.1 (Pin_1)
- net RS485_MAX485/B: now also J2.3 (Pin_3)
Changed lines of the file:
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@@
   (junction (at 240.03 46.482) (diameter 0) (color 0 0 0 0)
   )
-  (wire (pts (xy 234.315 127.635) (xy 238.76 127.635))
+  (wire (pts (xy 255.905 123.825) (xy 255.905 130.175))
     (stroke (width 0) (type default))
   )
@@
     (stroke (width 0) (type default))
   )
+  (wire (pts (xy 255.905 130.175) (xy 251.46 130.175))
+    (stroke (width 0) (type default))
+  )
   (wire (pts (xy 240.03 38.1) (xy 240.03 46.482))
     (stroke (width 0) (type default))
@@
     (stroke (width 0) (type default))
   )
+  (wire (pts (xy 255.905 136.525) (xy 255.905 132.715))
+    (stroke (width 0) (type default))
+  )
   (wire (pts (xy 160.02 110.49) (xy 186.69 110.49))
     (stroke (width 0) (type default))
@@
     (stroke (width 0) (type default))
   )
+  (wire (pts (xy 251.46 132.715) (xy 255.905 132.715))
+    (stroke (width 0) (type default))
+  )
   (wire (pts (xy 224.79 132.715) (xy 238.76 132.715))
     (stroke (width 0) (type default))
@@
   )
   (wire (pts (xy 83.82 111.125) (xy 115.57 111.125))
-    (stroke (width 0) (type default))
-  )
-  (wire (pts (xy 238.76 125.095) (xy 236.22 125.095))
-    (stroke (width 0) (type default))
-  )
-  (wire (pts (xy 236.22 125.095) (xy 236.22 117.475))
     (stroke (width 0) (type default))
   )
@@
     )
   )
-  (symbol (lib_id "power:GND") (at 234.315 127.635 270) (unit 1)
-    (in_bom yes) (on_board yes) (dnp no) (fields_autoplaced)
-    (property "Reference" "#PWR09" (at 227.965 127.635 0)
-      (effects (font (size 1.27 1.27)) hide)
-    )
-    (property "Value" "GND" (at 231.14 127.635 90)
-      (effects (font (size 1.27 1.27)) (justify right))
-    )
-    (property "Footprint" "" (at 234.315 127.635 0)
-      (effects (font (size 1.27 1.27)) hide)
-    )
-    (property "Datasheet" "" (at 234.315 127.635 0)
+  (symbol (lib_id "power:GND") (at 255.905 136.525 0) (unit 1)
+    (in_bom yes) (on_board yes) (dnp no) (fields_autoplaced)
+    (property "Reference" "#PWR09" (at 255.905 142.875 0)
+      (effects (font (size 1.27 1.27)) hide)
+    )
+    (property "Value" "GND" (at 255.905 140.97 0)
+      (effects (font (size 1.27 1.27)))
+    )
+    (property "Footprint" "" (at 255.905 136.525 0)
+      (effects (font (size 1.27 1.27)) hide)
+    )
+    (property "Datasheet" "" (at 255.905 136.525 0)
       (effects (font (size 1.27 1.27)) hide)
     )
@@
         (path "/b79ebed7-e146-448b-8dab-0aefb3e182ca/eafd7aad-682e-4ec9-bdb3-c64de2178f38"
           (reference "#PWR064") (unit 1)
+        )
+      )
+    )
+  )
+  (symbol (lib_id "Connector_Generic:Conn_02x02_Odd_Even") (at 243.84 130.175 0) (unit 1)
+    (in_bom yes) (on_board yes) (dnp no) (fields_autoplaced)
+    (property "Reference" "J2" (at 245.11 124.46 0)
+      (effects (font (size 1.27 1.27)))
+    )
+    (property "Value" "Conn_02x02_Odd_Even" (at 245.11 127 0)
+      (effects (font (size 1.27 1.27)))
+    )
+    (property "Footprint" "Connector_Molex:Molex_Mini-Fit_Jr_5569-04A2_2x02_P4.20mm_Horizontal" (at 243.84 130.175 0)
+      (effects (font (size 1.27 1.27)) hide)
+    )
+    (property "Datasheet" "~" (at 243.84 130.175 0)
+      (effects (font (size 1.27 1.27)) hide)
+    )
+    (pin "1")
+    (pin "2")
+    (pin "3")
+    (pin "4")
+    (instances
+      (project "GSM_module_v3"
+        (path "/8cb1db64-3fcc-4fb6-aa5a-7b4a50bb28df"
+          (reference "J2") (unit 1)
+        )
+      )
+      (project "BIM_PCB"
+        (path "/b79ebed7-e146-448b-8dab-0aefb3e182ca"
+          (reference "J6") (unit 1)
         )
       )
@@
     )
   )
-  (symbol (lib_id "power:+5V") (at 236.22 117.475 0) (unit 1)
-    (in_bom yes) (on_board yes) (dnp no) (fields_autoplaced)
-    (property "Reference" "#PWR061" (at 236.22 121.285 0)
-      (effects (font (size 1.27 1.27)) hide)
-    )
-    (property "Value" "+5V" (at 236.22 112.395 0)
-      (effects (font (size 1.27 1.27)))
-    )
-    (property "Footprint" "" (at 236.22 117.475 0)
-      (effects (font (size 1.27 1.27)) hide)
-    )
-    (property "Datasheet" "" (at 236.22 117.475 0)
+  (symbol (lib_id "power:+5V") (at 255.905 123.825 0) (unit 1)
+    (in_bom yes) (on_board yes) (dnp no) (fields_autoplaced)
+    (property "Reference" "#PWR061" (at 255.905 127.635 0)
+      (effects (font (size 1.27 1.27)) hide)
+    )
+    (property "Value" "+5V" (at 255.905 118.745 0)
+      (effects (font (size 1.27 1.27)))
+    )
+    (property "Footprint" "" (at 255.905 123.825 0)
+      (effects (font (size 1.27 1.27)) hide)
+    )
+    (property "Datasheet" "" (at 255.905 123.825 0)
       (effects (font (size 1.27 1.27)) hide)
     )
@@
         )
       )
-    )
-  )
-  (symbol (lib_id "Connector_Generic:Conn_01x04") (at 243.84 130.175 0) (mirror x) (unit 1)
-    (in_bom yes) (on_board yes) (dnp no)
-    (property "Reference" "J4" (at 247.015 130.175 0)
-      (effects (font (size 1.27 1.27)) (justify left))
-    )
-    (property "Value" "Conn_01x04" (at 247.015 127.635 0)
-      (effects (font (size 1.27 1.27)) (justify left))
-    )
-    (property "Footprint" "" (at 243.84 130.175 0)
-      (effects (font (size 1.27 1.27)) hide)
-    )
-    (property "Datasheet" "~" (at 243.84 130.175 0)
-      (effects (font (size 1.27 1.27)) hide)
-    )
-    (pin "1")
-    (pin "2")
-    (pin "3")
-    (pin "4")
-    (instances
-      (project "GSM_module_v3"
-        (path "/8cb1db64-3fcc-4fb6-aa5a-7b4a50bb28df"
-          (reference "J4") (unit 1)
-        )
-      )
