File: SRC/GPS_MODULE_V3/RS485_MAX485.kicad_sch (KiCad schematic)
At the start: 14 parts, among them U4 MAX485E, U5 TBU-CA065-200-WH, U6 TBU-CA065-200-WH

Commit message: layut completed
Parts:
- removed U5, U6: TBU-CA065-200-WH, Lib:TBU-CA065-200-WH, symbol MCD_General:TBU-CA065-200-WH
- added R28, R32: 0R, Resistor_SMD:R_0402_1005Metric, symbol Device:R_US
- D11, D12: value P0640TA -> BEP0080MA; footprint Diode_SMD:D_SMA -> Diode_SMD:D_SOD-123
Connections:
- net A: now also R32.2
- net B: now also R28.2
- net at D10.1 (K), R25.2, R27.2: now also R28.1
- net at D10.2 (K), R26.2, R27.1: now also R32.1
Other:
- moved on the sheet: D11
Changed lines of the file:
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@@
   (junction (at 135.255 91.44) (diameter 0) (color 0 0 0 0)
   )
-  (junction (at 188.595 87.63) (diameter 0) (color 0 0 0 0)
-  )
   (junction (at 120.65 99.06) (diameter 0) (color 0 0 0 0)
   )
@@
   )
   (junction (at 69.85 64.77) (diameter 0) (color 0 0 0 0)
+  )
+  (junction (at 180.34 87.63) (diameter 0) (color 0 0 0 0)
   )
   (junction (at 155.575 102.87) (diameter 0) (color 0 0 0 0)
@@
     (stroke (width 0) (type dash_dot))
   )
-  (wire (pts (xy 183.515 87.63) (xy 188.595 87.63))
+  (wire (pts (xy 167.005 87.63) (xy 180.34 87.63))
     (stroke (width 0) (type default))
   )
@@
     (stroke (width 0) (type default))
   )
-  (wire (pts (xy 188.595 116.84) (xy 194.945 116.84))
+  (wire (pts (xy 180.34 116.84) (xy 194.945 116.84))
     (stroke (width 0) (type default))
   )
@@
     (stroke (width 0) (type default))
   )
-  (wire (pts (xy 188.595 87.63) (xy 188.595 106.68))
+  (wire (pts (xy 180.34 87.63) (xy 180.34 106.68))
     (stroke (width 0) (type default))
   )
@@
     (stroke (width 0) (type default))
   )
-  (wire (pts (xy 188.595 114.3) (xy 188.595 116.84))
+  (wire (pts (xy 180.34 114.3) (xy 180.34 116.84))
     (stroke (width 0) (type default))
   )
@@
   )
   (wire (pts (xy 201.93 99.06) (xy 201.93 102.87))
+    (stroke (width 0) (type default))
+  )
+  (wire (pts (xy 180.34 87.63) (xy 201.93 87.63))
     (stroke (width 0) (type default))
   )
@@
     (stroke (width 0) (type default))
   )
-  (wire (pts (xy 183.515 102.87) (xy 201.93 102.87))
-    (stroke (width 0) (type default))
-  )
-  (wire (pts (xy 188.595 87.63) (xy 201.93 87.63))
+  (wire (pts (xy 167.005 102.87) (xy 201.93 102.87))
     (stroke (width 0) (type default))
   )
@@
     )
   )
+  (symbol (lib_id "Device:R_US") (at 163.195 87.63 90) (unit 1)
+    (in_bom yes) (on_board yes) (dnp no) (fields_autoplaced)
+    (property "Reference" "R28" (at 163.195 82.55 90)
+      (effects (font (size 1.27 1.27)))
+    )
+    (property "Value" "0R" (at 163.195 85.09 90)
+      (effects (font (size 1.27 1.27)))
+    )
+    (property "Footprint" "Resistor_SMD:R_0402_1005Metric" (at 163.449 86.614 90)
+      (effects (font (size 1.27 1.27)) hide)
+    )
+    (property "Datasheet" "~" (at 163.195 87.63 0)
+      (effects (font (size 1.27 1.27)) hide)
+    )
+    (pin "1")
+    (pin "2")
+    (instances
+      (project "GSM_module_v3"
+        (path "/8cb1db64-3fcc-4fb6-aa5a-7b4a50bb28df/10f6c1c7-c1fc-4fab-93e4-de442e304026"
+          (reference "R28") (unit 1)
+        )
+      )
+      (project "BIM_PCB"
+        (path "/b79ebed7-e146-448b-8dab-0aefb3e182ca/1465f310-1de3-424a-8f4a-a980ed628081"
+          (reference "R37") (unit 1)
+        )
+      )
+      (project "MAX485"
+        (path "/bc82bdd3-8c90-4895-abd4-de755b621eab"
+          (reference "R42") (unit 1)
+        )
+      )
+      (project "ELIESTER_V2"
+        (path "/efe55700-0211-4481-aa01-7a7eb74def17/d62e2e8a-503b-4c7c-a2bb-b074e6b71fb0"
+          (reference "R42") (unit 1)
+        )
+      )
+    )
+  )
   (symbol (lib_id "power:GND") (at 59.69 111.76 0) (unit 1)
     (in_bom yes) (on_board yes) (dnp no) (fields_autoplaced)
@@
         (path "/efe55700-0211-4481-aa01-7a7eb74def17/d62e2e8a-503b-4c7c-a2bb-b074e6b71fb0"
           (reference "#PWR088") (unit 1)
-        )
-      )
-    )
-  )
-  (symbol (lib_id "MCD_General:TBU-CA065-200-WH") (at 169.545 82.55 0) (unit 1)
-    (in_bom yes) (on_board yes) (dnp no) (fields_autoplaced)
-    (property "Reference" "U5" (at 171.45 81.915 0)
-      (effects (font (size 1.27 1.27)))
-    )
-    (property "Value" "TBU-CA065-200-WH" (at 171.45 84.455 0)
-      (effects (font (size 1.27 1.27)))
-    )
-    (property "Footprint" "Lib:TBU-CA065-200-WH" (at 169.545 83.82 0)
-      (effects (font (size 1.27 1.27)) hide)
-    )
-    (property "Datasheet" "" (at 169.545 83.82 0)
-      (effects (font (size 1.27 1.27)) hide)
-    )
-    (pin "1")
-    (pin "2")
-    (instances
-      (project "GSM_module_v3"
-        (path "/8cb1db64-3fcc-4fb6-aa5a-7b4a50bb28df/10f6c1c7-c1fc-4fab-93e4-de442e304026"
-          (reference "U5") (unit 1)
-        )
-      )
-      (project "BIM_PCB"
-        (path "/b79ebed7-e146-448b-8dab-0aefb3e182ca/1465f310-1de3-424a-8f4a-a980ed628081"
-          (reference "U4") (unit 1)
-        )
-      )
-      (project "MAX485"
-        (path "/bc82bdd3-8c90-4895-abd4-de755b621eab"
-          (reference "U13") (unit 1)
-        )
-      )
-      (project "ELIESTER_V2"
-        (path "/efe55700-0211-4481-aa01-7a7eb74def17/d62e2e8a-503b-4c7c-a2bb-b074e6b71fb0"
-          (reference "U13") (unit 1)
         )
       )
@@
     )
   )
-  (symbol (lib_id "MCD_General:TBU-CA065-200-WH") (at 169.545 97.79 0) (unit 1)
-    (in_bom yes) (on_board yes) (dnp no) (fields_autoplaced)
-    (property "Reference" "U6" (at 171.45 97.155 0)
-      (effects (font (size 1.27 1.27)))
-    )
-    (property "Value" "TBU-CA065-200-WH" (at 171.45 99.695 0)
-      (effects (font (size 1.27 1.27)))
-    )
-    (property "Footprint" "Lib:TBU-CA065-200-WH" (at 169.545 99.06 0)
-      (effects (font (size 1.27 1.27)) hide)
-    )
-    (property "Datasheet" "" (at 169.545 99.06 0)
-      (effects (font (size 1.27 1.27)) hide)
-    )
-    (pin "1")
-    (pin "2")
-    (instances
-      (project "GSM_module_v3"
-        (path "/8cb1db64-3fcc-4fb6-aa5a-7b4a50bb28df/10f6c1c7-c1fc-4fab-93e4-de442e304026"
-          (reference "U6") (unit 1)
-        )
-      )
-      (project "BIM_PCB"
-        (path "/b79ebed7-e146-448b-8dab-0aefb3e182ca/1465f310-1de3-424a-8f4a-a980ed628081"
-          (reference "U6") (unit 1)
-        )
-      )
-      (project "MAX485"
-        (path "/bc82bdd3-8c90-4895-abd4-de755b621eab"
-          (reference "U16") (unit 1)
-        )
-      )
-      (project "ELIESTER_V2"
-        (path "/efe55700-0211-4481-aa01-7a7eb74def17/d62e2e8a-503b-4c7c-a2bb-b074e6b71fb0"
-          (reference "U16") (unit 1)
-        )
-      )
-    )
-  )
   (symbol (lib_id "Device:C_Small") (at 59.69 59.69 0) (unit 1)
     (in_bom yes) (on_board yes) (dnp no) (fields_autoplaced)
@@
     )
   )
-  (symbol (lib_id "Diode:SD05_SOD323") (at 188.595 110.49 90) (unit 1)
-    (in_bom yes) (on_board yes) (dnp no) (fields_autoplaced)
-    (property "Reference" "D11" (at 191.135 109.855 90)
+  (symbol (lib_id "Diode:SD05_SOD323") (at 180.34 110.49 90) (unit 1)
+    (in_bom yes) (on_board yes) (dnp no) (fields_autoplaced)
+    (property "Reference" "D11" (at 183.515 109.855 90)
       (effects (font (size 1.27 1.27)) (justify right))
     )
-    (property "Value" "P0640TA" (at 191.135 112.395 90)
+    (property "Value" "BEP0080MA" (at 183.515 112.395 90)
       (effects (font (size 1.27 1.27)) (justify right))
     )
-    (property "Footprint" "Diode_SMD:D_SMA" (at 193.675 110.49 0)
-      (effects (font (size 1.27 1.27)) hide)
-    )
-    (property "Datasheet" "https://www.littelfuse.com/~/media/electronics/datasheets/tvs_diode_arrays/littelfuse_tvs_diode_array_sd_c_datasheet.pdf.pdf" (at 188.595 110.49 0)
+    (property "Footprint" "Diode_SMD:D_SOD-123" (at 185.42 110.49 0)
+      (effects (font (size 1.27 1.27)) hide)
+    )
+    (property "Datasheet" "https://www.littelfuse.com/~/media/electronics/datasheets/tvs_diode_arrays/littelfuse_tvs_diode_array_sd_c_datasheet.pdf.pdf" (at 180.34 110.49 0)
       (effects (font (size 1.27 1.27)) hide)
     )
@@
         (path "/8cb1db64-3fcc-4fb6-aa5a-7b4a50bb28df/10f6c1c7-c1fc-4fab-93e4-de442e304026"
           (reference "#PWR042") (unit 1)
+        )
+      )
+    )
+  )
+  (symbol (lib_id "Device:R_US") (at 163.195 102.87 90) (unit 1)
+    (in_bom yes) (on_board yes) (dnp no) (fields_autoplaced)
+    (property "Reference" "R32" (at 163.195 97.79 90)
+      (effects (font (size 1.27 1.27)))
+    )
+    (property "Value" "0R" (at 163.195 100.33 90)
+      (effects (font (size 1.27 1.27)))
+    )
+    (property "Footprint" "Resistor_SMD:R_0402_1005Metric" (at 163.449 101.854 90)
+      (effects (font (size 1.27 1.27)) hide)
+    )
+    (property "Datasheet" "~" (at 163.195 102.87 0)
+      (effects (font (size 1.27 1.27)) hide)
+    )
+    (pin "1")
+    (pin "2")
+    (instances
+      (project "GSM_module_v3"
+        (path "/8cb1db64-3fcc-4fb6-aa5a-7b4a50bb28df/10f6c1c7-c1fc-4fab-93e4-de442e304026"
+          (reference "R32") (unit 1)
+        )
+      )
+      (project "BIM_PCB"
+        (path "/b79ebed7-e146-448b-8dab-0aefb3e182ca/1465f310-1de3-424a-8f4a-a980ed628081"
+          (reference "R37") (unit 1)
+        )
+      )
+      (project "MAX485"
+        (path "/bc82bdd3-8c90-4895-abd4-de755b621eab"
+          (reference "R42") (unit 1)
+        )
+      )
+      (project "ELIESTER_V2"
+        (path "/efe55700-0211-4481-aa01-7a7eb74def17/d62e2e8a-503b-4c7c-a2bb-b074e6b71fb0"
+          (reference "R42") (unit 1)
         )
       )
@@
       (effects (font (size 1.27 1.27)) (justify right))
     )
-    (property "Value" "P0640TA" (at 204.47 112.395 90)
+    (property "Value" "BEP0080MA" (at 204.47 112.395 90)
       (effects (font (size 1.27 1.27)) (justify right))
     )
-    (property "Footprint" "Diode_SMD:D_SMA" (at 207.01 110.49 0)
-      (effects (font (size 1.27 1.27)) hide)
-    )
+    (property "Footprint" "Diode_SMD:D_SOD-123" (at 207.01 110.49 0)
+      (effects (font (size 1.27 1.27)) hide)
+    )
