File: SRC/GPS_MODULE_V3/SIM7000E_GPRS_SIM MODULE.kicad_sch (KiCad schematic)
At the start: 49 parts, among them J3 SIM_Card, Q5 BSN20, U3 SIM7000E

Commit message: layut completed
Parts:
- J3: value SIM_Card -> Micro_Sim_card; footprint Lib:GCT_SIM7100-6-1-15-00-A_REVC -> Lib:SMC2026; MPN (none) -> SMC-202-6
Changed lines of the file:
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@@
   (symbol (lib_id "Connector:SIM_Card") (at 31.75 170.18 0) (mirror y) (unit 1)
     (in_bom yes) (on_board yes) (dnp no) (fields_autoplaced)
-    (property "Reference" "J3" (at 29.21 157.48 0)
+    (property "Reference" "J3" (at 29.21 156.21 0)
       (effects (font (size 1.27 1.27)))
     )
-    (property "Value" "SIM_Card" (at 29.21 160.02 0)
+    (property "Value" "Micro_Sim_card" (at 29.21 158.75 0)
       (effects (font (size 1.27 1.27)))
     )
-    (property "Footprint" "Lib:GCT_SIM7100-6-1-15-00-A_REVC" (at 31.75 160.02 0)
+    (property "Footprint" "Lib:SMC2026" (at 31.75 160.02 0)
       (effects (font (size 1.27 1.27)) hide)
     )
-    (property "Datasheet" " ~" (at 27.94 157.48 0)
+    (property "Datasheet" "https://datasheet.lcsc.com/lcsc/2109061830_XUNPU-SMC-202-6_C266634.pdf" (at 27.94 157.48 0)
+      (effects (font (size 1.27 1.27)) hide)
+    )
+    (property "MPN" "SMC-202-6" (at 31.75 170.18 0)
       (effects (font (size 1.27 1.27)) hide)
     )
@@
     (pin "C2")
     (pin "C3")
-    (pin "C4")
     (pin "C5")
     (pin "C6")
     (pin "C7")
-    (pin "C8")
     (pin "MP1")
     (pin "MP2")
