File: SRC/GPS_MODULE_V3.kicad_pro/TF_CARD_CONN.kicad_sch (KiCad schematic)
At the start: 9 parts, among them J7 Micro_SD_Card

Commit message: routing
Changed lines of the file:
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@@
-    (effects (font (size 1.27 1.27)) (justify left bottom))
-  )
-  (label "2V8" (at 161.925 84.455 0) (fields_autoplaced)
     (effects (font (size 1.27 1.27)) (justify left bottom))
   )
@@
     (effects (font (size 1.27 1.27)) (justify left bottom))
   )
+  (hierarchical_label "2V8" (shape input) (at 161.925 84.455 90) (fields_autoplaced)
+    (effects (font (size 1.27 1.27)) (justify left))
+  )
   (hierarchical_label "SD_D0" (shape bidirectional) (at 196.215 112.395 180) (fields_autoplaced)
