File: SRC/GPS_MODULE_V3.kicad_pro/FLASH_MEMORY.kicad_sch (KiCad schematic)
At the start: 2 parts, among them U8 W25Q32JVSS

Commit message: completed GPS
Changed lines of the file:
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@@
     (effects (font (face "Agency FB") (size 5 5) (thickness 0.4) bold) (justify left bottom))
   )
-  (hierarchical_label "SCK" (shape input) (at 118.11 96.52 180) (fields_autoplaced)
-    (effects (font (size 1.27 1.27)) (justify right))
+  (hierarchical_label "SCK" (shape input) (at 118.11 96.52 0) (fields_autoplaced)
+    (effects (font (size 1.27 1.27)) (justify left))
   )
   (hierarchical_label "MISO" (shape bidirectional) (at 118.11 101.6 180) (fields_autoplaced)
