File: SRC/GPS_MODULE_V3.kicad_pro/MOSFET_LOGIC_LEVEL_TRANSLATOR.kicad_sch (KiCad schematic)
At the start: 20 parts, among them Q2 2N7002

Commit message: updates on BOM, CPL and gerbers
Parts:
- removed Q2 (x5): 2N7002, Package_TO_SOT_SMD:SOT-23, symbol Device:Q_NMOS_GSD
- removed R16 (x5): 1K, Resistor_SMD:R_0402_1005Metric, symbol Device:R_US
- removed R16 (x5), R17 (x5): 10K, Resistor_SMD:R_0402_1005Metric, symbol Device:R_US
- added Q2: 2N7002, Package_TO_SOT_SMD:SOT-23, symbol Device:Q_NMOS_GSD
- added R16, R17: 10K, Resistor_SMD:R_0402_1005Metric, symbol Device:R_US
- added R16: 1K, Resistor_SMD:R_0402_1005Metric, symbol Device:R_US
Connections:
- net HIGH_SIDE_POWER_LEVEL: now also R17.1
- net LOW_SIDE_POWER_LEVEL: now also Q2.1 (G), R16.1
- new net: Q2.2 (S), R16.2, R16.2
- new net HIGH_SIDE_LOGIC_SIGNAL: Q2.3 (D), R17.2
- new net LOW_SIDE_LOGIC_SIGNAL: R16.1
Other:
- note added: "HIGH LEVEL SIDE"
- note added: "LOW LEVEL SIDE"

Commit message: completed GPS ecoboda files
Parts:
- removed R16: 1K, Resistor_SMD:R_0402_1005Metric, symbol Device:R_US
Connections:
- net LOW_SIDE_LOGIC_SIGNAL: now also Q2.2 (S), R16.2
Changed lines of the file:
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@@
     (stroke (width 0) (type default))
   )
-  (wire (pts (xy 114.3 109.855) (xy 130.81 109.855))
+  (wire (pts (xy 92.71 109.855) (xy 130.81 109.855))
     (stroke (width 0) (type default))
   )
   (wire (pts (xy 130.81 109.855) (xy 140.97 109.855))
-    (stroke (width 0) (type default))
-  )
-  (wire (pts (xy 106.68 109.855) (xy 92.71 109.855))
     (stroke (width 0) (type default))
   )
@@
         )
       )
-    )
-  )
-  (symbol (lib_id "Device:R_US") (at 110.49 109.855 90) (unit 1)
-    (in_bom yes) (on_board yes) (dnp no) (fields_autoplaced)
-    (property "Reference" "R16" (at 110.49 105.41 90)
-      (effects (font (size 1.27 1.27)))
-    )
-    (property "Value" "1K" (at 110.49 107.95 90)
-      (effects (font (size 1.27 1.27)))
-    )
-    (property "Footprint" "Resistor_SMD:R_0402_1005Metric" (at 110.744 108.839 90)
-      (effects (font (size 1.27 1.27)) hide)
-    )
-    (property "Datasheet" "~" (at 110.49 109.855 0)
-      (effects (font (size 1.27 1.27)) hide)
-    )
-    (pin "1")
-    (pin "2")
-    (instances
-      (project "soilpal_v2_display"
-        (path "/0f8c6740-d040-4ce5-9b68-f1b365682d4f/882dd2d8-3941-4c8a-8503-e0fde4fea083/3e85a5a0-554b-44dc-a879-1e045818e6b3"
-          (reference "R16") (unit 1)
-        )
-        (path "/0f8c6740-d040-4ce5-9b68-f1b365682d4f/882dd2d8-3941-4c8a-8503-e0fde4fea083/b27c05a5-0db8-40ac-9faa-2b77abef5682"
-          (reference "R16") (unit 1)
-        )
-      )
-      (project "SmartCaravan"
-        (path "/7543dfcb-36f2-4cd3-8ba8-a9efbe7f97b6/4b192ea4-b50c-4f29-914a-cb19b995dc6c"
-          (reference "R16") (unit 1)
-        )
-        (path "/7543dfcb-36f2-4cd3-8ba8-a9efbe7f97b6/67648d4e-4082-43b9-a0d1-7155e8bb1efd"
-          (reference "R18") (unit 1)
-        )
-        (path "/7543dfcb-36f2-4cd3-8ba8-a9efbe7f97b6/ba1df6c2-c1e6-44ae-8b3d-dd996450ce77"
-          (reference "R20") (unit 1)
-        )
-        (path "/7543dfcb-36f2-4cd3-8ba8-a9efbe7f97b6/b4baabbf-1ea4-440a-9d55-ec64ff5e04c5"
-          (reference "R22") (unit 1)
-        )
-        (path "/7543dfcb-36f2-4cd3-8ba8-a9efbe7f97b6/7c63ae45-86df-4e05-bfa9-a69699819595"
-          (reference "R24") (unit 1)
-        )
-        (path "/7543dfcb-36f2-4cd3-8ba8-a9efbe7f97b6/e935d23e-356e-4ed7-923e-4ff3e9d1207b"
-          (reference "R26") (unit 1)
-        )
-      )
-      (project "GSM_GPRS_MODULE_SIM7000G"
-        (path "/7b5c61bb-3beb-4d85-afc0-546a503e9b5f/3e85a5a0-554b-44dc-a879-1e045818e6b3"
-          (reference "R16") (unit 1)
-        )
-        (path "/7b5c61bb-3beb-4d85-afc0-546a503e9b5f/b27c05a5-0db8-40ac-9faa-2b77abef5682"
-          (reference "R16") (unit 1)
-        )
-      )
-      (project "GPS_MODULE_V3.kicad_pro"
-        (path "/8cb1db64-3fcc-4fb6-aa5a-7b4a50bb28df/bf84f6a6-afcd-4d16-b49e-82022456ea82/e4c474fa-b78e-4e69-8a10-750455b88e98"
-          (reference "R33") (unit 1)
-        )
-        (path "/8cb1db64-3fcc-4fb6-aa5a-7b4a50bb28df/bf84f6a6-afcd-4d16-b49e-82022456ea82/9af48e8e-497e-49d4-800c-d02a4a3413ff"
-          (reference "R36") (unit 1)
-        )
-        (path "/8cb1db64-3fcc-4fb6-aa5a-7b4a50bb28df/bf84f6a6-afcd-4d16-b49e-82022456ea82/6f7505d4-6bef-405c-a8b0-f60f4ef1ff15"
-          (reference "R45") (unit 1)
-        )
-        (path "/8cb1db64-3fcc-4fb6-aa5a-7b4a50bb28df/bf84f6a6-afcd-4d16-b49e-82022456ea82/3afb6843-ee45-474d-abc0-9babe8038f58"
-          (reference "R50") (unit 1)
-        )
-      )
-      (project "BIM_PCB"
-        (path "/b79ebed7-e146-448b-8dab-0aefb3e182ca/2c1557a8-70b5-4535-b084-9e551cb55dcd/edbaae4f-de44-432d-a3ab-ffa1b686e8fe"
-          (reference "R19") (unit 1)
-        )
-        (path "/b79ebed7-e146-448b-8dab-0aefb3e182ca/2c1557a8-70b5-4535-b084-9e551cb55dcd/7d84c724-e693-4753-b610-031b5bfcbd41"
-          (reference "R50") (unit 1)
-        )
-        (path "/b79ebed7-e146-448b-8dab-0aefb3e182ca/2c1557a8-70b5-4535-b084-9e551cb55dcd/0c226a2b-7062-4290-934f-18e7ef8514ce"
-          (reference "R53") (unit 1)
-        )
-        (path "/b79ebed7-e146-448b-8dab-0aefb3e182ca/2c1557a8-70b5-4535-b084-9e551cb55dcd/592382d8-1d8e-43ab-883d-cb4e58136da0"
-          (reference "R56") (unit 1)
-        )
-      )
-      (project "BI_DIRECTIONAL_LOGIC_LEVEL_TRANSLATOR_MOSFET-use"
-        (path "/d5ed9ea7-1d20-4cba-b955-75adcb1b4a20"
-          (reference "R16") (unit 1)
-        )
-      )
-      (project "ELIESTER_V2"
-        (path "/efe55700-0211-4481-aa01-7a7eb74def17/414f1577-4ce3-43d7-bbf4-7827eef840c4/b27c05a5-0db8-40ac-9faa-2b77abef5682"
-          (reference "R76") (unit 1)
-        )
-        (path "/efe55700-0211-4481-aa01-7a7eb74def17/414f1577-4ce3-43d7-bbf4-7827eef840c4/3e85a5a0-554b-44dc-a879-1e045818e6b3"
-          (reference "R69") (unit 1)
-        )
-      )
