File: SRC/GPS_MODULE_V3.kicad_pro/RS485_MAX485.kicad_sch (KiCad schematic)
At the start: 14 parts, among them U4 MAX485E

Commit message: GPS all files BOM and placemnt guide files added
Parts:
- removed R28, R32: 0R, Resistor_SMD:R_0402_1005Metric, symbol Device:R_US
- added L5, L6: L_Ferrite, Inductor_SMD:L_0402_1005Metric, symbol Device:L_Ferrite
Connections:
- net A: now also L6.2
- net B: now also L5.2
- net at D10.1 (K), R25.2, R27.2: now also L5.1
- net at D10.2 (K), R26.2, R27.1: now also L6.1
Changed lines of the file:
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@@
-    )
-  )
-  (symbol (lib_id "Device:R_US") (at 163.195 87.63 90) (unit 1)
-    (in_bom yes) (on_board yes) (dnp no) (fields_autoplaced)
-    (property "Reference" "R28" (at 163.195 82.55 90)
-      (effects (font (size 1.27 1.27)))
-    )
-    (property "Value" "0R" (at 163.195 85.09 90)
-      (effects (font (size 1.27 1.27)))
-    )
-    (property "Footprint" "Resistor_SMD:R_0402_1005Metric" (at 163.449 86.614 90)
-      (effects (font (size 1.27 1.27)) hide)
-    )
-    (property "Datasheet" "~" (at 163.195 87.63 0)
-      (effects (font (size 1.27 1.27)) hide)
-    )
-    (pin "1")
-    (pin "2")
-    (instances
-      (project "GPS_MODULE_V3.kicad_pro"
-        (path "/8cb1db64-3fcc-4fb6-aa5a-7b4a50bb28df/10f6c1c7-c1fc-4fab-93e4-de442e304026"
-          (reference "R28") (unit 1)
-        )
-      )
-      (project "BIM_PCB"
-        (path "/b79ebed7-e146-448b-8dab-0aefb3e182ca/1465f310-1de3-424a-8f4a-a980ed628081"
-          (reference "R37") (unit 1)
-        )
-      )
-      (project "MAX485"
-        (path "/bc82bdd3-8c90-4895-abd4-de755b621eab"
-          (reference "R42") (unit 1)
-        )
-      )
-      (project "ELIESTER_V2"
-        (path "/efe55700-0211-4481-aa01-7a7eb74def17/d62e2e8a-503b-4c7c-a2bb-b074e6b71fb0"
-          (reference "R42") (unit 1)
-        )
-      )
     )
   )
@@
     )
   )
+  (symbol (lib_id "Device:L_Ferrite") (at 163.195 87.63 90) (unit 1)
+    (in_bom yes) (on_board yes) (dnp no) (fields_autoplaced)
+    (property "Reference" "L5" (at 163.195 80.8774 90)
+      (effects (font (size 1.27 1.27)))
+    )
+    (property "Value" "L_Ferrite" (at 163.195 83.4174 90)
+      (effects (font (size 1.27 1.27)))
+    )
+    (property "Footprint" "Inductor_SMD:L_0402_1005Metric" (at 163.195 87.63 0)
+      (effects (font (size 1.27 1.27)) hide)
+    )
+    (property "Datasheet" "~" (at 163.195 87.63 0)
+      (effects (font (size 1.27 1.27)) hide)
+    )
+    (pin "1")
+    (pin "2")
+    (instances
+      (project "GPS_MODULE_V3.kicad_pro"
+        (path "/8cb1db64-3fcc-4fb6-aa5a-7b4a50bb28df/10f6c1c7-c1fc-4fab-93e4-de442e304026"
+          (reference "L5") (unit 1)
+        )
+      )
+    )
+  )
   (symbol (lib_id "Diode:SD05_SOD323") (at 180.34 110.49 90) (unit 1)
     (in_bom yes) (on_board yes) (dnp no) (fields_autoplaced)
@@
         (path "/8cb1db64-3fcc-4fb6-aa5a-7b4a50bb28df/10f6c1c7-c1fc-4fab-93e4-de442e304026"
           (reference "#PWR042") (unit 1)
-        )
-      )
-    )
-  )
-  (symbol (lib_id "Device:R_US") (at 163.195 102.87 90) (unit 1)
-    (in_bom yes) (on_board yes) (dnp no) (fields_autoplaced)
-    (property "Reference" "R32" (at 163.195 97.79 90)
-      (effects (font (size 1.27 1.27)))
-    )
-    (property "Value" "0R" (at 163.195 100.33 90)
-      (effects (font (size 1.27 1.27)))
-    )
-    (property "Footprint" "Resistor_SMD:R_0402_1005Metric" (at 163.449 101.854 90)
-      (effects (font (size 1.27 1.27)) hide)
-    )
-    (property "Datasheet" "~" (at 163.195 102.87 0)
-      (effects (font (size 1.27 1.27)) hide)
-    )
-    (pin "1")
-    (pin "2")
-    (instances
-      (project "GPS_MODULE_V3.kicad_pro"
-        (path "/8cb1db64-3fcc-4fb6-aa5a-7b4a50bb28df/10f6c1c7-c1fc-4fab-93e4-de442e304026"
-          (reference "R32") (unit 1)
-        )
-      )
-      (project "BIM_PCB"
-        (path "/b79ebed7-e146-448b-8dab-0aefb3e182ca/1465f310-1de3-424a-8f4a-a980ed628081"
-          (reference "R37") (unit 1)
-        )
-      )
-      (project "MAX485"
-        (path "/bc82bdd3-8c90-4895-abd4-de755b621eab"
-          (reference "R42") (unit 1)
-        )
-      )
-      (project "ELIESTER_V2"
-        (path "/efe55700-0211-4481-aa01-7a7eb74def17/d62e2e8a-503b-4c7c-a2bb-b074e6b71fb0"
-          (reference "R42") (unit 1)
         )
       )
@@
         )
       )
+    )
+  )
+  (symbol (lib_id "Device:L_Ferrite") (at 163.195 102.87 90) (unit 1)
+    (in_bom yes) (on_board yes) (dnp no) (fields_autoplaced)
+    (property "Reference" "L6" (at 163.195 96.1174 90)
+      (effects (font (size 1.27 1.27)))
+    )
+    (property "Value" "L_Ferrite" (at 163.195 98.6574 90)
+      (effects (font (size 1.27 1.27)))
+    )
+    (property "Footprint" "Inductor_SMD:L_0402_1005Metric" (at 163.195 102.87 0)
+      (effects (font (size 1.27 1.27)) hide)
+    )
+    (property "Datasheet" "~" (at 163.195 102.87 0)
+      (effects (font (size 1.27 1.27)) hide)
+    )
+    (pin "1")
+    (pin "2")
+    (instances
+      (project "GPS_MODULE_V3.kicad_pro"
+        (path "/8cb1db64-3fcc-4fb6-aa5a-7b4a50bb28df/10f6c1c7-c1fc-4fab-93e4-de442e304026"
+          (reference "L6") (unit 1)
+        )
+      )
