File: SRC/GPS_MODULE_V3.kicad_pro/SY8089_BUCK_CONVERTER.kicad_sch (KiCad schematic)
At the start: 12 parts, among them U1 SY8089AAAC

Commit message: GPS all files BOM and placemnt guide files added
Parts:
- C38: footprint Capacitor_SMD:C_0603_1608Metric -> Capacitor_SMD:C_0402_1005Metric
- TP2: footprint TestPoint:TestPoint_Pad_D1.5mm -> TestPoint:TestPoint_Pad_D1.0mm
Changed lines of the file:
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@@
       (effects (font (size 1.27 1.27)) (justify left))
     )
-    (property "Footprint" "Capacitor_SMD:C_0603_1608Metric" (at 105.41 93.98 0)
+    (property "Footprint" "Capacitor_SMD:C_0402_1005Metric" (at 105.41 93.98 0)
       (effects (font (size 1.27 1.27)) hide)
     )
@@
       (effects (font (size 1.27 1.27)) (justify left) hide)
     )
-    (property "Footprint" "TestPoint:TestPoint_Pad_D1.5mm" (at 208.915 83.82 0)
-      (effects (font (size 1.27 1.27)) hide)
-    )
+    (property "Footprint" "TestPoint:TestPoint_Pad_D1.0mm" (at 208.915 83.82 0)
+      (effects (font (size 1.27 1.27)) hide)
+    )
